File: TimedTrigger.kicad_pcb (KiCad board)
At the start: 2 copper layers, 100 x 60 mm, 84 parts, among them J1 9V_JACK, J10 Trigger_PHNX, J2 PWR_IN_PHNX, J3 OUT1_PHNX, J4 OUT1_3.5mm, J5 OUT2_PHNX, J6 OUT2_3.5mm, J7 OUT3_PHNX, J8 OUT3_3.5mm, J9 TRIGGER_3.5mm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

Commit message: Started laying out components
Parts:
- BT1: moved to B.Cu
- D4: value TIM1_IND -> TIM2_IND
- D5: value TIM1_IND -> TIM3_IND
- D6: value TIM1_IND -> THRESH_IND
- D7: value TIM1_IND -> INPUT_IND
- D8: value TIM1_IND -> TRIG_IND
- moved J10 167.6 mm to (67.0, 58.0), turned to 180 degrees
- moved J3 157.6 mm to (87.0, 58.0), turned to 180 degrees
- moved D1 152.7 mm to (132.5, 90.5), turned to 180 degrees
- moved R1 116.4 mm to (141.0, 98.5)
- moved J9 108.3 mm to (75.0, 59.0)
- moved J8 100.8 mm to (135.0, 59.0)
- moved J5 95.1 mm to (107.0, 58.0), turned to 180 degrees
- moved J4 94.8 mm to (95.0, 59.0)
- moved BT1 92.6 mm to (111.0, 79.0)
- moved J6 79.9 mm to (115.0, 59.0)
- moved J7 73.5 mm to (127.0, 58.0), turned to 180 degrees
- moved D2 39.1 mm to (141.0, 95.5)
- moved J1 5.66 mm to (136.0, 79.0)
- moved J2 4.61 mm to (141.5, 68.0)
- moved RV4 4.47 mm to (52.0, 86.0)
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Routing:
- added copper zone on B.Cu, net GND
- added copper zone on F.Cu, net GND
Other:
- board text added: "ON←POWER→OFF"
- board text added: "◀OUT1▼"
- board text added: "◀OUT2▼"
- board text added: "◀OUT3▼"
- board text added: "◀TRIG IN▼"
